File: Kicad_Schematic/block_diagram/led_strip.kicad_sch (KiCad schematic)
At the start: 6 parts

Commit message: edited block diagrams from design rev 2
Connections:
- net GND: now reaches addressable_led1. (Dout), addressable_led2. (Dout)
- net GND: now also addressable_led3. (Dout)
- new net: addressable_led1. (Dout), addressable_led2. (Dout)
- new net: addressable_led2. (Dout), addressable_led3. (Dout)
- new net 5V: addressable_led1. (Dout), addressable_led2. (Dout), addressable_led3. (Dout)
Other:
- note added: "From Pico GND"
- note added: "From Pico GPIO Pin"
- note removed: "To Pico GND"
Changed lines of the file:
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@@
 	(text "From buck converter\n"
 		(exclude_from_sim no)
-		(at 88.9 76.2 0)
+		(at 78.232 76.2 0)
 		(effects
 			(font
@@
 		)
 	)
-	(text "To Pico GND\n"
-		(exclude_from_sim no)
-		(at 83.82 100.33 0)
+	(text "From Pico GND\n"
+		(exclude_from_sim no)
+		(at 76.454 99.822 0)
+		(effects
+			(font
+				(size 1.27 1.27)
+			)
+		)
+	)
+	(text "From Pico GPIO Pin\n"
+		(exclude_from_sim no)
+		(at 78.232 87.63 0)
 		(effects
 			(font
@@
 	)
 	(junction
+		(at 140.97 97.79)
+		(diameter 0)
+		(color 0 0 0 0)
+	)
+	(junction
 		(at 88.9 77.47)
 		(diameter 0)
@@
 	)
 	(junction
+		(at 140.97 77.47)
+		(diameter 0)
+		(color 0 0 0 0)
+	)
+	(junction
 		(at 115.57 97.79)
 		(diameter 0)
@@
 	(wire
 		(pts
-			(xy 78.74 77.47) (xy 88.9 77.47)
-		)
-		(stroke
-			(width 0)
-			(type default)
-		)
-	)
-	(wire
-		(pts
-			(xy 78.74 97.79) (xy 88.9 97.79)
-		)
-		(stroke
-			(width 0)
-			(type default)
-		)
-	)
-	(wire
-		(pts
 			(xy 115.57 77.47) (xy 140.97 77.47)
 		)
@@
 	(wire
 		(pts
+			(xy 67.31 97.79) (xy 88.9 97.79)
+		)
+		(stroke
+			(width 0)
+			(type default)
+		)
+	)
+	(wire
+		(pts
 			(xy 140.97 77.47) (xy 140.97 85.09)
 		)
@@
 	(wire
 		(pts
+			(xy 67.31 88.9) (xy 88.9 88.9)
+		)
+		(stroke
+			(width 0)
+			(type default)
+		)
+	)
+	(wire
+		(pts
+			(xy 140.97 77.47) (xy 166.37 77.47)
+		)
+		(stroke
+			(width 0)
+			(type default)
+		)
+	)
+	(wire
+		(pts
 			(xy 88.9 77.47) (xy 115.57 77.47)
 		)
@@
 	(wire
 		(pts
+			(xy 67.31 77.47) (xy 88.9 77.47)
+		)
+		(stroke
+			(width 0)
+			(type default)
+		)
+	)
+	(wire
+		(pts
+			(xy 140.97 97.79) (xy 166.37 97.79)
+		)
+		(stroke
+			(width 0)
+			(type default)
+		)
+	)
+	(wire
+		(pts
 			(xy 140.97 97.79) (xy 140.97 92.71)
 		)
@@
 			(width 0)
 			(type default)
+		)
+	)
+	(global_label "5V"
+		(shape input)
+		(at 67.31 77.47 180)
+		(fields_autoplaced yes)
+		(effects
+			(font
+				(size 1.27 1.27)
+			)
+			(justify right)
+		)
+		(property "Intersheetrefs" "${INTERSHEET_REFS}"
+			(at 62.0267 77.47 0)
+			(effects
+				(font
+					(size 1.27 1.27)
+				)
+				(justify right)
+				(hide yes)
+			)
 		)
 	)
@@
 					(unit 1)
 				)
+			)
+		)
+	)
+	(symbol
+		(lib_id "power:GND")
+		(at 67.31 97.79 0)
+		(unit 1)
+		(exclude_from_sim no)
+		(in_bom yes)
+		(on_board yes)
+		(dnp no)
+		(fields_autoplaced yes)
+		(property "Reference" "#PWR04"
+			(at 67.31 104.14 0)
+			(effects
+				(font
+					(size 1.27 1.27)
+				)
+				(hide yes)
+			)
+		)
+		(property "Value" "GND"
+			(at 67.31 102.87 0)
+			(effects
+				(font
+					(size 1.27 1.27)
+				)
+			)
+		)
+		(property "Footprint" ""
+			(at 67.31 97.79 0)
+			(effects
+				(font
+					(size 1.27 1.27)
+				)
+				(hide yes)
+			)
+		)
+		(property "Datasheet" ""
+			(at 67.31 97.79 0)
+			(effects
+				(font
+					(size 1.27 1.27)
+				)
+				(hide yes)
+			)
+		)
+		(property "Description" "Power symbol creates a global label with name \"GND\" , ground"
+			(at 67.31 97.79 0)
+			(effects
+				(font
+					(size 1.27 1.27)
+				)
+				(hide yes)
+			)
+		)
+		(pin "1"
+		)
+		(instances
+			(project ""
+				(path "/7a474c3b-855e-4a89-97e9-3d42055b899d/66bf6c33-5aac-4565-8433-307d195f0022"
+					(reference "#PWR04")
+					(unit 1)
+				)
